File: pciex1-m2-cm4g.kicad_pcb (KiCad board)
At the start: 2 copper layers, 35 x 104.4 mm, 18 parts, among them J1 Bus_M.2_Socket_M, J2 Bus_PCI_Express_x1, J3 Bus_PCI_Express_x1, J4 Bus_PCI_Express_x1, J5 PROTO6x17

Commit message: added SUSClk
Parts:
- added C7: 100n, Capacitor_SMD:C_1206_3216Metric, F.Cu at (133.7, 125.1)
- added X1: 32.768kHz, Oscillator:Oscillator_SMD_EuroQuartz_XO32-4Pin_3.2x2.5mm, F.Cu at (129.7, 125.6)
- moved C6 3.04 mm to (131.2, 121.1), turned to 0 degrees
- moved R1 0.75 mm to (131.7, 129.6)
Connections:
- J1 pad 68: unconnected-(J1-SUSCLK-Pad68) -> Net-(J1-SUSCLK)
Routing:
- net Net-(J1-SUSCLK): track 0.00 -> 26.0 mm, vias 0 -> 2
- net +3.3V: track 221.0 -> 228.9 mm
